File: diff_tran.kicad_pcb (KiCad board)
At the start: 2 copper layers, 28.7 x 13.8 mm, 29 parts, among them IC1 SN65LVDM176, IC2 SN65LVDM176, IC3 SN65LVDM176, IC4 SN65LVDM176, J1 SOLDER_JUMPER, J10 SOLDER_JUMPER, J11 SOLDER_JUMPER, J12 SOLDER_JUMPER, J2 SOLDER_JUMPER, J3 SOLDER_JUMPER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

Commit message: Tracks
Parts:
- added ?: , LercheTech:Lerche_via_0.35_GND_MaskOver, F.Cu at (146.2, 98.9)
- moved R3 4.65 mm to (151.2, 96.9), turned to 90 degrees
- moved R4 4.53 mm to (151.2, 99.5), turned to 270 degrees
- moved R2 4.37 mm to (151.2, 94.4), turned to 270 degrees
- moved R5 4.34 mm to (151.3, 102.0), turned to 90 degrees
- moved J10 2.12 mm to (149.7, 96.9), turned to 270 degrees
- moved J11 1.73 mm to (149.7, 99.5), turned to 90 degrees
- moved J9 1.24 mm to (149.7, 94.4), turned to 90 degrees
- moved J12 0.67 mm to (149.7, 102.0), turned to 270 degrees
Connections:
- J12 pad 1: Net-(IC1-Pad7) -> Net-(IC1-Pad6)
- R5 pad 2: Net-(IC1-Pad6) -> Net-(IC1-Pad7)
Routing:
- net +3V3: track 0.00 -> 53.9 mm, vias 0 -> 1
- net MISO: track 0.00 -> 30.9 mm
- net MOSI: track 0.00 -> 18.5 mm
- net Net-(IC3-Pad6): track 0.00 -> 13.8 mm
- net Net-(IC4-Pad6): track 0.00 -> 13.7 mm
- net Net-(IC2-Pad6): track 0.00 -> 13.7 mm
- net Net-(IC1-Pad6): track 0.00 -> 13.5 mm
- net Net-(IC1-Pad7): track 0.00 -> 11.5 mm
- net Net-(IC2-Pad7): track 0.00 -> 11.0 mm
- net GND: track 0.00 -> 10.6 mm
- net Net-(IC3-Pad7): track 0.00 -> 10.2 mm
- net Net-(IC4-Pad7): track 0.00 -> 10.1 mm
- net SCK: track 0.00 -> 6.84 mm
- net SSEL: track 0.00 -> 5.83 mm
- net Net-(D1-Pad2): track 0.00 -> 2.20 mm
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Other:
- net class Default: clearance 0.2 -> 0.16; trace_width 0.25 -> 0.2
- rule trace_clearance: 0.2 -> 0.16
- rule trace_min: 0.2 -> 0.15

Commit message: Commit
Connections:
- IC1 pad 1: SCK -> SSEL
- IC1 pad 4: SCK -> SSEL
- IC2 pad 1: MOSI -> MISO
- IC2 pad 4: MOSI -> MISO
- IC3 pad 1: MISO -> MOSI
- IC3 pad 4: MISO -> MOSI
- IC4 pad 1: SSEL -> SCK
- IC4 pad 4: SSEL -> SCK
Routing:
- net MISO: track 30.9 -> 12.0 mm
- net MOSI: track 18.5 -> 11.9 mm
- net SSEL: track 5.83 -> 11.8 mm
- net SCK: track 6.84 -> 12.1 mm
- net +3V3: track 53.9 -> 56.7 mm, vias 1 -> 2

Commit message: Added some text, almost finished
Added some text, almost finished
Parts:
- added ?: , LercheTech:Lerche_via_0.35_GND_MaskOver, F.Cu at (142.5, 103.0)
- added ?: , LercheTech:Lerche_via_0.35_GND_MaskOver, F.Cu at (155.0, 100.6)
- added ?: , LercheTech:Lerche_via_0.35_GND_MaskOver, F.Cu at (148.9, 103.2)
- added ?: , LercheTech:Lerche_via_0.35_GND_MaskOver, F.Cu at (148.6, 100.9)
- added ?: , LercheTech:Lerche_via_0.35_GND_MaskOver, F.Cu at (148.9, 98.2)
- added ?: , LercheTech:Lerche_via_0.35_GND_MaskOver, F.Cu at (148.5, 95.5)
- added ?: , LercheTech:Lerche_via_0.35_GND_MaskOver, F.Cu at (147.3, 92.3)
- added ?: , LercheTech:Lerche_via_0.35_GND_MaskOver, F.Cu at (143.8, 90.7)
- added ?: , LercheTech:Lerche_via_0.35_GND_MaskOver, F.Cu at (143.8, 92.5)
- added ?: , LercheTech:Lerche_via_0.35_GND_MaskOver, F.Cu at (142.7, 93.7)
- added ?: , LercheTech:Lerche_via_0.35_GND_MaskOver, F.Cu at (141.2, 93.1)
- added ?: , LercheTech:Lerche_via_0.35_GND_MaskOver, F.Cu at (152.6, 97.9)
- added ?: , LercheTech:Lerche_via_0.35_GND_MaskOver, F.Cu at (142.2, 98.8)
- added ?: , LercheTech:Lerche_via_0.35_GND_MaskOver, F.Cu at (142.5, 100.8)
- added ?: , LercheTech:Lerche_via_0.35_GND_MaskOver, F.Cu at (136.2, 93.8)
- added ?: , LercheTech:Lerche_via_0.35_GND_MaskOver, F.Cu at (132.7, 101.3)
- added ?: , LercheTech:Lerche_via_0.35_GND_MaskOver, F.Cu at (134.2, 103.1)
- added ?: , LercheTech:Lerche_via_0.35_GND_MaskOver, F.Cu at (140.3, 103.1)
- added ?: , LercheTech:Lerche_via_0.35_GND_MaskOver, F.Cu at (139.7, 101.6)
- added ?: , LercheTech:Lerche_via_0.35_GND_MaskOver, F.Cu at (139.3, 98.3)
- added ?: , LercheTech:Lerche_via_0.35_GND_MaskOver, F.Cu at (134.0, 98.1)
- added ?: , LercheTech:Lerche_via_0.35_GND_MaskOver, F.Cu at (139.7, 94.0)
- added ?: , LercheTech:Lerche_via_0.35_GND_MaskOver, F.Cu at (152.5, 93.3)
- added ?: , LercheTech:Lerche_via_0.35_GND_MaskOver, F.Cu at (134.3, 93.1)
- added ?: , LercheTech:Lerche_via_0.35_GND_MaskOver, F.Cu at (148.9, 92.6)
- added ?: , LercheTech:Lerche_via_0.35_GND_MaskOver, F.Cu at (151.2, 91.6)
- added ?: , LercheTech:Lerche_via_0.35_GND_MaskOver, F.Cu at (157.5, 93.1)
- added ?: , LercheTech:Lerche_via_0.35_GND_MaskOver, F.Cu at (155.1, 93.1)
- added ?: , LercheTech:Lerche_via_0.35_GND_MaskOver, F.Cu at (157.4, 95.6)
- added ?: , LercheTech:Lerche_via_0.35_GND_MaskOver, F.Cu at (157.4, 98.1)
Routing:
- net +3V3: track 56.7 -> 72.8 mm, vias 2 -> 3
Other:
- board text added: "3V3"
- board text added: "DE"
- board text added: "GND"
- board text added: "MISO"
- board text added: "MOSI"
- board text added: "SCK"
- board text added: "SSEL"
- board text added: "~RE"
