File: diff_tran.sch (KiCad schematic (older format))
At the start: 29 parts, among them IC1 SN65LVDM176, IC2 SN65LVDM176, IC3 SN65LVDM176, IC4 SN65LVDM176, J1 SOLDER_JUMPER, J10 SOLDER_JUMPER, J11 SOLDER_JUMPER, J12 SOLDER_JUMPER, J2 SOLDER_JUMPER, J3 SOLDER_JUMPER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

Commit message: Added some text, almost finished
Added some text, almost finished
Connections:
- net MISO: now also IC2.1 (R), IC2.4 (D); no longer IC3.1 (R), IC3.4 (D)
- net MOSI: now also IC3.1 (R), IC3.4 (D); no longer IC2.1 (R), IC2.4 (D)
- net SCK: now also IC4.1 (R), IC4.4 (D); no longer IC1.1 (R), IC1.4 (D)
- net SSEL: now also IC1.1 (R), IC1.4 (D); no longer IC4.1 (R), IC4.4 (D)
Changed lines of the file:
@@
 LIBS:valves
 LIBS:lerchetech
+LIBS:diff_tran-cache
 EELAYER 25 0
 EELAYER END
@@
 Text GLabel 2850 2800 2    39   Output ~ 0
 SCK
+Text GLabel 4550 5000 0    39   Input ~ 0
+SCK
+Text GLabel 4550 4400 0    39   Input ~ 0
+MOSI
+Text GLabel 4550 3500 0    39   Output ~ 0
+MISO
 Text GLabel 4550 3200 0    39   Input ~ 0
-SCK
-Text GLabel 4550 3800 0    39   Input ~ 0
-MOSI
-Text GLabel 4550 4100 0    39   Output ~ 0
-MISO
-Text GLabel 4550 5000 0    39   Input ~ 0
 SSEL
 $Comp
@@
 	1    0    0    -1
 $EndComp
+Text GLabel 4550 4700 0    39   Output ~ 0
+SCK
+Text GLabel 4550 4100 0    39   Output ~ 0
+MOSI
+Text GLabel 4550 3800 0    39   Input ~ 0
+MISO
 Text GLabel 4550 2900 0    39   Output ~ 0
-SCK
-Text GLabel 4550 3500 0    39   Output ~ 0
-MOSI
-Text GLabel 4550 4400 0    39   Input ~ 0
-MISO
-Text GLabel 4550 4700 0    39   Output ~ 0
 SSEL
 $Comp
